File: 12.kicad_sch (KiCad schematic)
At the start: 59 parts, among them P1 TSW-107-08-G-D, P6 M20-9990346, U1 SN74AVC4T245PW, U2 SN74AVC4T245PW, U27 SN74AVC4T245PW, U37 CD74HC4024PWR, U38 74HCT151D,652, U39 SN74AVC4T245PW, U4 24LC32A-I/ST, U40 24LC32A-I/ST

Commit message: update
Parts:
- added P10, P8, P9: JMP2, Custom:JMP_Custom, symbol Custom:JMP2
- added P14, P15, P17: JMP, Custom:JMP_Custom, symbol Custom:JMP
- C1, C110, C112, C13, C14, C150, C151, C152, C153, C154, C163, C164, C2, C3, C59, C6: footprint Capacitor_SMD:C_0603_1608Metric -> Custom:C_0603_1608Metric
- R13, R138, R14, R15, R16, R161, R162, R21, R23, R25, R26, R27, R28, R30, R31, R32, R5, R6, R7, R8, R94: footprint Resistor_SMD:R_0603_1608Metric -> Custom:R_0603_1608Metric
- U1, U2, U27, U39: footprint Package_SO:TSSOP-16-1EP_4.4x5mm_P0.65mm_EP3x3mm -> Package_SO:TSSOP-16_4.4x5mm_P0.65mm
Connections:
- net A0: now also P10.2
- net A1: now also P9.2
- net A2: now also P8.2
- net AGND: now also P10.1, P8.1, P9.1; no longer U1.17 (EP), U2.17 (EP), U27.17 (EP), U39.17 (EP)
- net BURST_1V8: now also P15.1; no longer P1.3
- net MUXOUT_1V8: now also P17.2; no longer P1.2
- net TXDATA_1V8: now also P14.1; no longer P1.1
- new net: P1.3, P15.2
- new net: P1.1, P14.2
- new net: P1.2, P17.1
