File: 6.kicad_sch (KiCad schematic)
At the start: 20 parts, among them T1 TC1-1-13M+, T3 TC1-1-13M+, U14 LTC5548IUDB#TRPBF, U6 LTC5548IUDB#TRPBF

Commit message: update
Parts:
- C23, C27, C78, C88: footprint Capacitor_SMD:C_0603_1608Metric -> Custom:C_0603_1608Metric
Connections:
- net VDD_3V3: now reaches C78.1, C88.1, U14.7 (EN), U14.9 (VCC)
- net VDD_3V3: now also C23.1, C27.1, U6.7 (EN), U6.9 (VCC)
Changed lines of the file:
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@@
 	)
 	(junction
+		(at 179.07 106.172)
+		(diameter 0)
+		(color 0 0 0 0)
+	)
+	(junction
 		(at 261.874 175.514)
 		(diameter 0)
@@
 	)
 	(junction
+		(at 179.07 208.026)
+		(diameter 0)
+		(color 0 0 0 0)
+	)
+	(junction
 		(at 167.64 120.904)
 		(diameter 0)
@@
 	(wire
 		(pts
+			(xy 179.07 106.172) (xy 186.944 106.172)
+		)
+		(stroke
+			(width 0)
+			(type default)
+		)
+	)
+	(wire
+		(pts
 			(xy 294.14 172.212) (xy 292.862 172.212)
 		)
@@
 	(wire
 		(pts
-			(xy 167.64 208.026) (xy 167.64 209.804)
-		)
-		(stroke
-			(width 0)
-			(type default)
-		)
-	)
-	(wire
-		(pts
 			(xy 167.64 106.172) (xy 167.64 107.95)
 		)
@@
 	(wire
 		(pts
-			(xy 179.07 106.172) (xy 179.07 107.95)
-		)
-		(stroke
-			(width 0)
-			(type default)
-		)
-	)
-	(wire
-		(pts
 			(xy 139.7 172.466) (xy 139.7 174.752)
 		)
@@
 	(wire
 		(pts
-			(xy 104.394 199.644) (xy 106.934 199.644)
+			(xy 182.88 208.026) (xy 179.07 208.026)
 		)
 		(stroke
@@
 	(wire
 		(pts
-			(xy 146.558 172.466) (xy 146.558 178.816)
+			(xy 104.394 199.644) (xy 106.934 199.644)
 		)
 		(stroke
@@
 	(wire
 		(pts
-			(xy 188.468 91.694) (xy 188.468 92.964)
+			(xy 146.558 172.466) (xy 146.558 178.816)
 		)
 		(stroke
@@
 	(wire
 		(pts
-			(xy 167.64 198.882) (xy 167.64 208.026)
+			(xy 188.468 91.694) (xy 188.468 92.964)
 		)
 		(stroke
@@
 	(wire
 		(pts
-			(xy 179.07 208.026) (xy 179.07 209.804)
+			(xy 167.64 198.882) (xy 167.64 208.026)
 		)
 		(stroke
@@
 	(wire
 		(pts
+			(xy 167.64 208.026) (xy 167.64 209.804)
+		)
+		(stroke
+			(width 0)
+			(type default)
+		)
+	)
+	(wire
+		(pts
 			(xy 124.46 199.136) (xy 124.46 201.676)
 		)
@@
 	(wire
 		(pts
+			(xy 179.07 106.172) (xy 179.07 107.95)
+		)
+		(stroke
+			(width 0)
+			(type default)
+		)
+	)
+	(wire
+		(pts
 			(xy 264.16 175.514) (xy 265.684 175.514)
 		)
@@
 	(wire
 		(pts
+			(xy 179.07 208.026) (xy 179.07 209.804)
+		)
+		(stroke
+			(width 0)
+			(type default)
+		)
+	)
+	(wire
+		(pts
 			(xy 291.6 70.358) (xy 292.862 70.358)
 		)
@@
 		)
 	)
+	(global_label "VDD_3V3"
+		(shape input)
+		(at 182.88 208.026 0)
+		(fields_autoplaced yes)
+		(effects
+			(font
+				(size 1.27 1.27)
+			)
+			(justify left)
+		)
+		(property "Intersheetrefs" "${INTERSHEET_REFS}"
+			(at 193.969 208.026 0)
+			(effects
+				(font
+					(size 1.27 1.27)
+				)
+				(justify left)
+				(hide yes)
+			)
+		)
+	)
 	(global_label "RF_IO_0"
 		(shape input)
@@
 		)
 	)
+	(global_label "VDD_3V3"
+		(shape input)
+		(at 186.944 106.172 0)
+		(fields_autoplaced yes)
+		(effects
+			(font
+				(size 1.27 1.27)
+			)
+			(justify left)
+		)
+		(property "Intersheetrefs" "${INTERSHEET_REFS}"
+			(at 198.033 106.172 0)
+			(effects
+				(font
+					(size 1.27 1.27)
+				)
+				(justify left)
+				(hide yes)
+			)
+		)
+	)
 	(global_label "LO_IN_1"
 		(shape input)
@@
 			)
 		)
-		(property "Footprint" "Capacitor_SMD:C_0603_1608Metric"
+		(property "Footprint" "Custom:C_0603_1608Metric"
 			(at 166.878 200.406 0)
 			(effects
@@
 			)
 		)
-		(property "Footprint" "Capacitor_SMD:C_0603_1608Metric"
+		(property "Footprint" "Custom:C_0603_1608Metric"
 			(at 178.308 98.552 0)
 			(effects
@@
 			)
 		)
-		(property "Footprint" "Capacitor_SMD:C_0603_1608Metric"
+		(property "Footprint" "Custom:C_0603_1608Metric"
 			(at 166.878 98.552 0)
 			(effects
@@
 			)
 		)
-		(property "Footprint" "Capacitor_SMD:C_0603_1608Metric"
+		(property "Footprint" "Custom:C_0603_1608Metric"
 			(at 178.308 200.406 0)
 			(effects
