File: 7.kicad_sch (KiCad schematic)
At the start: 28 parts, among them P12 36900000, P13 36900000, P19 36900000, P4 36900000, P5 36900000, P7 36900000, T2 TC1-1-13M+, U10 ADRF5019BCPZN, U12 HMC654LP2E, U13 ADL8107ACPZN, U7 LTC5548IUDB#TRPBF

Commit message: update
Parts:
- C76, C83, C86, C87, C9: footprint Capacitor_SMD:C_0603_1608Metric -> Custom:C_0603_1608Metric
- R124, R164, R91: footprint Resistor_SMD:R_0603_1608Metric -> Custom:R_0603_1608Metric
Changed lines of the file:
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@@
 			)
 		)
-		(property "Footprint" "Capacitor_SMD:C_0603_1608Metric"
+		(property "Footprint" "Custom:C_0603_1608Metric"
 			(at 176.53 138.938 0)
 			(effects
@@
 			)
 		)
-		(property "Footprint" "Capacitor_SMD:C_0603_1608Metric"
+		(property "Footprint" "Custom:C_0603_1608Metric"
 			(at 258.064 73.406 0)
 			(effects
@@
 			)
 		)
-		(property "Footprint" "Capacitor_SMD:C_0603_1608Metric"
+		(property "Footprint" "Custom:C_0603_1608Metric"
 			(at 372.364 90.424 0)
 			(effects
@@
 			)
 		)
-		(property "Footprint" "Capacitor_SMD:C_0603_1608Metric"
+		(property "Footprint" "Custom:C_0603_1608Metric"
 			(at 186.944 138.938 0)
 			(effects
@@
 			)
 		)
-		(property "Footprint" "Capacitor_SMD:C_0603_1608Metric"
+		(property "Footprint" "Custom:C_0603_1608Metric"
 			(at 250.952 86.36 0)
 			(effects
@@
 			)
 		)
-		(property "Footprint" "Resistor_SMD:R_0603_1608Metric"
+		(property "Footprint" "Custom:R_0603_1608Metric"
 			(at 295.91 197.866 0)
 			(effects
@@
 			)
 		)
-		(property "Footprint" "Resistor_SMD:R_0603_1608Metric"
+		(property "Footprint" "Custom:R_0603_1608Metric"
 			(at 209.55 99.568 0)
 			(effects
@@
 			)
 		)
-		(property "Footprint" "Resistor_SMD:R_0603_1608Metric"
+		(property "Footprint" "Custom:R_0603_1608Metric"
 			(at 260.35 171.704 0)
 			(effects
