File: 9.kicad_sch (KiCad schematic)
At the start: 34 parts, among them J10 0853050232, J3 0853050232, J4 0853050232, J5 0853050232, J6 0853050232, J7 0853050232, J8 0853050232, J9 0853050232, U23 ADRF5019BCPZN, U24 ADRF5019BCPZN, U25 EP2C+, U26 EP2C+

Commit message: update
Parts:
- C10, C109: footprint Capacitor_SMD:C_0603_1608Metric -> Custom:C_0603_1608Metric
Changed lines of the file:
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@@
 			)
 		)
-		(property "Footprint" "Capacitor_SMD:C_0603_1608Metric"
+		(property "Footprint" "Custom:C_0603_1608Metric"
 			(at 44.45 98.298 0)
 			(effects
@@
 			)
 		)
-		(property "Footprint" "Capacitor_SMD:C_0603_1608Metric"
+		(property "Footprint" "Custom:C_0603_1608Metric"
 			(at 211.836 147.32 0)
 			(effects
