File: 10.kicad_sch (KiCad schematic)
At the start: 92 parts, among them P16 632723300011, U11 ADM7170ACPZ-4.2-R7, U28 ADM7170ACPZ-4.2-R7, U29 ADM7150ACPZ-1.8-R7, U30 LT3460ESC6#TRMPBF, U31 ADP7158ARDZ-3.3-R7, U32 ADP7118AUJZ-R7, U35 ADM7150ACPZ-1.8-R7, U36 LTC4217HFE#PBF

Commit message: update
Parts:
- C114, C115, C116, C117, C118, C119, C121, C122, C123, C124, C125, C126, C127, C128, C129, C130, C135, C137, C138, C140, C141, C143, C144, C145, C146, C147, C148, C170, C171, C172, C173, C174, C175, C48, C66, C68: footprint Capacitor_SMD:C_0603_1608Metric -> Custom:C_0603_1608Metric
- R10, R100, R101, R102, R11, R111, R12, R137, R139, R148, R149, R151, R152, R153, R156, R160, R17, R18, R19, R24, R50, R51, R53, R54, R57, R58, R59, R60, R61, R86, R88, R9, R92, R98, R99: footprint Resistor_SMD:R_0603_1608Metric -> Custom:R_0603_1608Metric
- R143: footprint Resistor_SMD:R_0603_1608Metric -> Custom:R_0402_1005Metric
Connections:
- net AGND: no longer U36.21 (PAD)
- net at R137.2, U36.1 (SENSE), U36.10 (SENSE)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: now also U36.21 (PAD)

Commit message: update
Parts:
- U36: footprint Package_SO:HTSSOP-20-1EP_4.4x6.5mm_P0.65mm_EP3.4x6.5mm_Mask2.4x3.7mm -> Custom:HTSSOP-20-1EP_4.4x6.5mm_P0.65mm_EP3.4x6.5mm_Mask2.4x3.7mm
Connections:
- net VSOURCE: now also C115.1, R148.1
Changed lines of the file:
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@@
 	)
 	(junction
+		(at 30.988 226.822)
+		(diameter 0)
+		(color 0 0 0 0)
+	)
+	(junction
 		(at 152.146 252.222)
 		(diameter 0)
@@
 	)
 	(junction
+		(at 30.988 232.664)
+		(diameter 0)
+		(color 0 0 0 0)
+	)
+	(junction
 		(at 69.342 252.73)
 		(diameter 0)
@@
 	(wire
 		(pts
+			(xy 30.988 226.822) (xy 52.324 226.822)
+		)
+		(stroke
+			(width 0)
+			(type default)
+		)
+	)
+	(wire
+		(pts
 			(xy 273.05 218.186) (xy 288.036 218.186)
 		)
@@
 	(wire
 		(pts
+			(xy 30.988 226.822) (xy 30.988 232.664)
+		)
+		(stroke
+			(width 0)
+			(type default)
+		)
+	)
+	(wire
+		(pts
 			(xy 115.316 240.792) (xy 115.316 235.712)
 		)
@@
 	(wire
 		(pts
-			(xy 37.084 226.822) (xy 52.324 226.822)
+			(xy 28.702 226.822) (xy 30.988 226.822)
 		)
 		(stroke
@@
 	(wire
 		(pts
-			(xy 25.4 232.664) (xy 37.846 232.664)
+			(xy 25.4 232.664) (xy 30.988 232.664)
 		)
 		(stroke
@@
 	(wire
 		(pts
+			(xy 30.988 232.664) (xy 37.846 232.664)
+		)
+		(stroke
+			(width 0)
+			(type default)
+		)
+	)
+	(wire
+		(pts
 			(xy 187.706 37.084) (xy 187.706 47.498)
 		)
@@
 	(global_label "VSOURCE"
 		(shape input)
-		(at 37.084 226.822 180)
+		(at 28.702 226.822 180)
 		(fields_autoplaced yes)
 		(effects
@@
 		)
 		(property "Intersheetrefs" "${INTERSHEET_REFS}"
-			(at 25.4507 226.822 0)
+			(at 17.0687 226.822 0)
 			(effects
 				(font
@@
 			)
 		)
-		(property "Footprint" "Package_SO:HTSSOP-20-1EP_4.4x6.5mm_P0.65mm_EP3.4x6.5mm_Mask2.4x3.7mm"
+		(property "Footprint" "Custom:HTSSOP-20-1EP_4.4x6.5mm_P0.65mm_EP3.4x6.5mm_Mask2.4x3.7mm"
 			(at 139.7 37.084 0)
 			(effects
