File: 11.kicad_sch (KiCad schematic)
At the start: 34 parts, among them P18 MTSW-107-07-T-S-240, P2 NPTC202KFMS-RC, P3 M20-9990246, U3 AD7291BCPZ

Commit message: update
Parts:
- added W1, W2, W3, W4, W5, W6, W7: ~, Custom:CPnt, symbol Custom:CPnt
- C169, C4, C5, C7, C8: footprint Capacitor_SMD:C_0603_1608Metric -> Custom:C_0603_1608Metric
- P2: footprint Connector_PinSocket_2.54mm:PinSocket_2x20_P2.54mm_Vertical_SMD -> Custom:PinSocket_2x20_P2.54mm_Vertical_SMD
- R1, R136, R190, R192, R2, R20, R22, R29, R55, R56, R62, R71, R72, R73, R74, R75, R76, R77, R78, R85, R97: footprint Resistor_SMD:R_0603_1608Metric -> Custom:R_0603_1608Metric
Connections:
- net IMON: now also W7.1
- net VDD_1V8: now also W6.1
- net VDD_3V0: now also W5.1
- net VDD_3V3: now also W3.1
- net VDD_4V5: now also W1.1
- net VDD_AMP: now also W2.1
- net VINPUT: now also W4.1
Other:
- moved on the sheet: R74

Commit message: update
Connections:
- net SD_RPI: now also R56.1, S3.2
Changed lines of the file:
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@@
+	)
+	(junction
+		(at 122.428 216.154)
+		(diameter 0)
+		(color 0 0 0 0)
 	)
 	(junction
@@
 	(wire
 		(pts
-			(xy 122.428 212.852) (xy 122.428 221.488)
+			(xy 122.428 212.852) (xy 122.428 216.154)
 		)
 		(stroke
@@
 	(wire
 		(pts
+			(xy 118.364 216.154) (xy 122.428 216.154)
+		)
+		(stroke
+			(width 0)
+			(type default)
+		)
+	)
+	(wire
+		(pts
 			(xy 335.788 87.122) (xy 335.788 84.836)
 		)
@@
 	(wire
 		(pts
+			(xy 122.428 216.154) (xy 122.428 221.488)
+		)
+		(stroke
+			(width 0)
+			(type default)
+		)
+	)
+	(wire
+		(pts
 			(xy 291.846 119.38) (xy 291.846 137.414)
 		)
@@
 			(effects
 				(font
+					(size 1.27 1.27)
+				)
+				(justify right)
+				(hide yes)
+			)
+		)
+	)
+	(global_label "SD_RPI"
+		(shape input)
+		(at 118.364 216.154 180)
+		(fields_autoplaced yes)
+		(effects
+			(font
+				(size 1.27 1.27)
+			)
+			(justify right)
+		)
+		(property "Intersheetrefs" "${INTERSHEET_REFS}"
+			(at 108.7869 216.154 0)
+			(effects
+				(font
