File: 8.kicad_sch (KiCad schematic)
At the start: 53 parts, among them U33 HMC652LP2E, U34 HMC735LP5E, U5 ADF4159CCPZ, Y1 CWX823-100.0M

Commit message: update
Parts:
- C108, C11, C17, C19, C72: footprint Capacitor_SMD:C_0603_1608Metric -> Custom:C_0603_1608Metric
- R41: footprint Resistor_SMD:R_0603_1608Metric -> Custom:R_0603_1608Metric
Changed lines of the file:
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@@
 			)
 		)
-		(property "Footprint" "Capacitor_SMD:C_0603_1608Metric"
+		(property "Footprint" "Custom:C_0603_1608Metric"
 			(at 175.768 227.076 0)
 			(effects
@@
 			)
 		)
-		(property "Footprint" "Resistor_SMD:R_0603_1608Metric"
+		(property "Footprint" "Custom:R_0603_1608Metric"
 			(at 105.664 46.482 0)
 			(effects
@@
 			)
 		)
-		(property "Footprint" "Capacitor_SMD:C_0603_1608Metric"
+		(property "Footprint" "Custom:C_0603_1608Metric"
 			(at 104.902 65.024 0)
 			(effects
@@
 			)
 		)
-		(property "Footprint" "Capacitor_SMD:C_0603_1608Metric"
+		(property "Footprint" "Custom:C_0603_1608Metric"
 			(at 293.37 109.22 0)
 			(effects
@@
 			)
 		)
-		(property "Footprint" "Capacitor_SMD:C_0603_1608Metric"
+		(property "Footprint" "Custom:C_0603_1608Metric"
 			(at 133.858 100.584 0)
 			(effects
@@
 			)
 		)
-		(property "Footprint" "Capacitor_SMD:C_0603_1608Metric"
+		(property "Footprint" "Custom:C_0603_1608Metric"
 			(at 264.414 174.752 0)
 			(effects

Commit message: update
Connections:
- net VDD_4V75: no longer C134.1
- net at U34.19 (RFOUT): now also C134.1
Other:
- moved on the sheet: C134, U33
Changed lines of the file:
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@@
 	)
 	(junction
-		(at 275.844 229.108)
+		(at 273.812 234.442)
 		(diameter 0)
 		(color 0 0 0 0)
@@
 	)
 	(junction
-		(at 276.606 229.108)
+		(at 274.574 234.442)
 		(diameter 0)
 		(color 0 0 0 0)
@@
 	)
 	(junction
-		(at 279.146 229.108)
+		(at 277.114 234.442)
 		(diameter 0)
 		(color 0 0 0 0)
@@
 	)
 	(junction
-		(at 281.686 229.108)
+		(at 279.654 234.442)
 		(diameter 0)
 		(color 0 0 0 0)
@@
 	)
 	(junction
-		(at 241.554 216.916)
-		(diameter 0)
-		(color 0 0 0 0)
-	)
-	(junction
 		(at 213.36 115.316)
 		(diameter 0)
@@
 	(wire
 		(pts
-			(xy 297.434 216.916) (xy 292.354 216.916)
+			(xy 295.402 222.25) (xy 290.322 222.25)
 		)
 		(stroke
@@
 	(wire
 		(pts
-			(xy 279.146 229.108) (xy 281.686 229.108)
+			(xy 277.114 234.442) (xy 279.654 234.442)
 		)
 		(stroke
@@
 	(wire
 		(pts
+			(xy 247.142 222.25) (xy 235.966 222.25)
+		)
+		(stroke
+			(width 0)
+			(type default)
+		)
+	)
+	(wire
+		(pts
 			(xy 45.212 49.53) (xy 57.404 49.53)
 		)
@@
 	(wire
 		(pts
-			(xy 265.684 216.916) (xy 256.794 216.916)
+			(xy 263.652 222.25) (xy 254.762 222.25)
 		)
 		(stroke
@@
 	(wire
 		(pts
-			(xy 241.554 179.832) (xy 241.554 216.916)
+			(xy 241.554 179.832) (xy 241.554 217.043)
 		)
 		(stroke
@@
 	(wire
 		(pts
-			(xy 275.844 229.108) (xy 276.606 229.108)
+			(xy 273.812 234.442) (xy 274.574 234.442)
 		)
 		(stroke
@@
 	(wire
 		(pts
-			(xy 274.066 229.108) (xy 275.844 229.108)
+			(xy 272.034 234.442) (xy 273.812 234.442)
 		)
 		(stroke
@@
 	(wire
 		(pts
-			(xy 249.174 216.916) (xy 241.554 216.916)
-		)
-		(stroke
-			(width 0)
-			(type default)
-		)
-	)
-	(wire
-		(pts
 			(xy 265.176 179.832) (xy 265.176 184.15)
 		)
@@
 	(wire
 		(pts
-			(xy 275.844 231.902) (xy 275.844 229.108)
+			(xy 273.812 237.236) (xy 273.812 234.442)
 		)
 		(stroke
@@
 	(wire
 		(pts
-			(xy 281.686 229.108) (xy 284.226 229.108)
+			(xy 279.654 234.442) (xy 282.194 234.442)
 		)
 		(stroke
@@
 	(wire
 		(pts
-			(xy 241.554 216.916) (xy 241.554 217.043)
-		)
-		(stroke
-			(width 0)
-			(type default)
-		)
-	)
-	(wire
-		(pts
 			(xy 259.842 114.554) (xy 266.192 114.554)
 		)
@@
 	(wire
 		(pts
-			(xy 276.606 229.108) (xy 279.146 229.108)
+			(xy 274.574 234.442) (xy 277.114 234.442)
 		)
 		(stroke
@@
 	(global_label "LO_LOC"
 		(shape input)
-		(at 297.434 216.916 0)
+		(at 295.402 222.25 0)
 		(fields_autoplaced yes)
 		(effects
@@
 		)
 		(property "Intersheetrefs" "${INTERSHEET_REFS}"
-			(at 307.374 216.916 0)
+			(at 305.342 222.25 0)
 			(effects
 				(font
@@
 	(symbol
 		(lib_id "PABA-DP:GRM033R71A103KA01D")
-		(at 246.634 218.186 90)
+		(at 244.602 223.52 90)
 		(unit 1)
 		(exclude_from_sim no)
@@
 		(dnp no)
 		(property "Reference" "C134"
-			(at 248.666 218.694 90)
+			(at 246.634 224.028 90)
 			(effects
 				(font
@@
 		)
 		(property "Value" "GRM033R71A103KA01D"
-			(at 241.3 217.678 0)
+			(at 239.268 223.012 0)
 			(effects
 				(font
@@
 		)
 		(property "Footprint" "Capacitor_SMD:C_0201_0603Metric"
-			(at 239.776 217.678 0)
+			(at 237.744 223.012 0)
 			(effects
 				(font
@@
 		)
 		(property "Datasheet" "https://search.murata.co.jp/Ceramy/image/img/A01X/G101/ENG/GRM033R71A103KA01-01.pdf"
-			(at 237.236 218.44 0)
+			(at 235.204 223.774 0)
 			(effects
 				(font
@@
 		)
 		(property "Description" "10000 pF ±10% 10V Ceramic Capacitor X7R 0201 (0603 Metric)"
-			(at 265.43 217.678 0)
+			(at 263.398 223.012 0)
 			(effects
 				(font
@@
 		)
 		(property "C" "0.01uF"
-			(at 257.556 218.694 90)
+			(at 255.524 224.028 90)
 			(effects
 				(font
@@
 		)
 		(property "V" "10V"
-			(at 257.556 221.234 90)
+			(at 255.524 226.568 90)
 			(effects
 				(font
@@
 		)
 		(property "Acc" "10%"
-			(at 246.634 218.186 0)
+			(at 244.602 223.52 0)
 			(effects
 				(font
@@
 	(symbol
 		(lib_id "PABA-DP:HMC652LP2E")
-		(at 274.066 210.058 0)
+		(at 272.034 215.392 0)
 		(mirror y)
 		(unit 1)
@@
 		(dnp no)
 		(property "Reference" "U33"
-			(at 274.066 210.058 0)
+			(at 272.034 215.392 0)
 			(effects
 				(font
@@
 		)
 		(property "Value" "HMC652LP2E"
-			(at 274.574 211.836 0)
+			(at 272.542 217.17 0)
 			(effects
 				(font
@@
 		)
 		(property "Footprint" "Custom:HMC652LP2E TDFN 2x2"
-			(at 274.066 210.058 0)
+			(at 272.034 215.392 0)
 			(effects
 				(font
@@
 		)
 		(property "Datasheet" "https://www.analog.com/media/en/technical-documentation/data-sheets/hmc652lp2-hmc655lp2.pdf"
-			(at 274.066 210.058 0)
+			(at 272.034 215.392 0)
 			(effects
 				(font
@@
 		)
 		(property "Description" "RF Attenuators 2dB 0 Hz ~ 25 GHz 50 Ohms 6-TDFN Exposed Pad"
-			(at 274.066 210.058 0)
+			(at 272.034 215.392 0)
 			(effects
 				(font
@@
 	(symbol
 		(lib_id "PABA-DP:GND")
-		(at 275.844 231.902 0)
+		(at 273.812 237.236 0)
 		(unit 1)
 		(exclude_from_sim no)
@@
 		(dnp no)
 		(property "Reference" "#PWR0179"
-			(at 275.844 238.252 0)
+			(at 273.812 243.586 0)
 			(effects
 				(font
@@
 		)
 		(property "Value" "AGND"
-			(at 278.892 234.696 0)
+			(at 276.86 240.03 0)
 			(effects
 				(font
@@
 		)
 		(property "Footprint" ""
-			(at 275.844 231.902 0)
+			(at 273.812 237.236 0)
 			(effects
 				(font
@@
 		)
 		(property "Datasheet" ""
-			(at 275.844 231.902 0)
+			(at 273.812 237.236 0)
 			(effects
 				(font
@@
 		)
 		(property "Description" "Power symbol creates a global label with name \"GND\" , ground"
-			(at 275.844 231.902 0)
+			(at 273.812 237.236 0)
 			(effects
 				(font
